File: Philly_Node.kicad_sch (KiCad schematic)
At the start: 77 parts, among them J2 LED, J4 USB_C_Receptacle_USB2.0, J5 Multi, Q1 Q_Dual_NMOS_G1S2G2D2S1D1, Q4 Q_NMOS_GSD, SW2 D0, U1 BQ25176JDSGR, U2 MDBT50Q-U1MV2, U3 E22-900M22S, U4 TPS2120YFPR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

Commit message: Beginning of board adjustments to use multiple fabs.
Parts:
- C1, C2, C3: LCSC C19666 -> (none); MFR_NUM (none) -> CL10A475KO8NNNC
- C10, C13, C6, C8: LCSC C1525 -> (none); MFR_NUM (none) -> CL05B104KO5NNNC
- C4, C5: LCSC C1547 -> (none); MFR_NUM (none) -> CC0402JPNPO9BN120
- D4: renamed from D2; value LESD5D5_0CT1G -> ESD5Z5.0C; LCSC C383211 -> (none); MFR_NUM (none) -> ESD5Z5.0C
- D4: renamed from D5; value LESD5D5_0CT1G -> ESD5Z5.0C; LCSC C383211 -> (none); MFR_NUM (none) -> ESD5Z5.0C
- D4: value LESD5D5_0CT1G -> ESD5Z5.0C; LCSC C383211 -> (none); MFR_NUM (none) -> ESD5Z5.0C
- D4: renamed from D1; value LESD5D5_0CT1G -> ESD5Z5.0C; LCSC C383211 -> (none); MFR_NUM (none) -> ESD5Z5.0C
- D4: renamed from D3; value LESD5D5_0CT1G -> ESD5Z5.0C; LCSC C383211 -> (none); MFR_NUM (none) -> ESD5Z5.0C
- J4: MFR (none) -> Amphenol; MFR_NUM (none) -> GSB1C41110SSHR
- LED1, LED2: value MHPA1010RGBDT -> L201DS-QEPGBG2S; footprint Philly_Lib:LED-ARRAY-SMD_4P-L1.0-W1.0-TR-RD -> Philly_Lib:L201DS-QEPGBG2S; LCSC Part C404280 -> (none)
- SOL1: renamed from BAT1; LCSC C968533 -> (none); MF_NUM (none) -> S2B-PH-SM4-TB(LF)(SN)
- SOL1: LCSC C47647 -> (none); MFR (none) -> JST; MF_NUM (none) -> S2B-PH-SM4-TB(LF)(SN)
- Y1: MFR (none) -> Epson; MFR_NUM (none) -> FC3215AN 32.768K-C5NN60KC5
Changed lines of the file:
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@@
 			)
 		)
-		(property "LCSC" "C19666"
+		(property "MFR_NUM" "CL10A475KO8NNNC"
 			(at 127 27.94 0)
 			(effects
@@
 		(dnp no)
 		(fields_autoplaced yes)
-		(property "Reference" "D2"
+		(property "Reference" "D4"
 			(at 29.21 24.13 0)
 			(effects
@@
 			)
 		)
-		(property "Value" "LESD5D5_0CT1G"
+		(property "Value" "ESD5Z5.0C"
 			(at 29.21 26.67 0)
 			(effects
@@
 			)
 		)
-		(property "LCSC" "C383211"
+		(property "MFR_NUM" "ESD5Z5.0C"
 			(at 29.21 15.24 0)
 			(effects
@@
 			(project "Philly_Node"
 				(path "/14b26dc5-70cb-4d13-ac9b-7e033bbb860b"
-					(reference "D2")
+					(reference "D4")
 					(unit 1)
 				)
@@
 			)
 		)
-		(property "LCSC" "C19666"
+		(property "MFR_NUM" "CL10A475KO8NNNC"
 			(at 140.97 27.94 0)
 			(effects
@@
 			)
 		)
-		(property "LCSC" "C19666"
+		(property "MFR_NUM" "CL10A475KO8NNNC"
 			(at 149.86 41.91 0)
 			(effects
@@
 		(dnp no)
 		(fields_autoplaced yes)
-		(property "Reference" "D5"
+		(property "Reference" "D4"
 			(at 29.21 54.61 0)
 			(effects
@@
 			)
 		)
-		(property "Value" "LESD5D5_0CT1G"
+		(property "Value" "ESD5Z5.0C"
 			(at 29.21 57.15 0)
 			(effects
@@
 			)
 		)
-		(property "LCSC" "C383211"
+		(property "MFR_NUM" "ESD5Z5.0C"
 			(at 29.21 45.72 0)
 			(effects
@@
 			(project "Philly_Node"
 				(path "/14b26dc5-70cb-4d13-ac9b-7e033bbb860b"
-					(reference "D5")
+					(reference "D4")
 					(unit 1)
 				)
@@
 			)
 		)
-		(property "Value" "MHPA1010RGBDT"
+		(property "Value" "L201DS-QEPGBG2S"
 			(at 247.65 53.465 90)
 			(effects
@@
 			)
 		)
-		(property "Footprint" "Philly_Lib:LED-ARRAY-SMD_4P-L1.0-W1.0-TR-RD"
+		(property "Footprint" "Philly_Lib:L201DS-QEPGBG2S"
 			(at 228.6 50.8 0)
 			(effects
@@
 			)
 		)
-		(property "Datasheet" "https://lcsc.com/product-detail/Light-Emitting-Diodes-LED_MEIHUA-MHPA1010RGBDT_C404280.html"
+		(property "Datasheet" ""
 			(at 226.06 50.8 0)
 			(effects
@@
 			)
 		)
-		(property "LCSC Part" "C404280"
-			(at 223.52 50.8 0)
-			(effects
-				(font
-					(size 1.27 1.27)
-				)
-				(hide yes)
-			)
-		)
 		(property "Note" "Up Firing USER"
 			(at 247.65 53.34 90)
@@
 			)
 		)
-		(property "LCSC" "C1547"
+		(property "MFR_NUM" "CC0402JPNPO9BN120"
 			(at 171.45 67.31 90)
 			(effects
@@
 			)
 		)
-		(property "Value" "LESD5D5_0CT1G"
+		(property "Value" "ESD5Z5.0C"
 			(at 29.21 46.99 0)
 			(effects
@@
 			)
 		)
-		(property "LCSC" "C383211"
+		(property "MFR_NUM" "ESD5Z5.0C"
 			(at 29.21 35.56 0)
 			(effects
@@
 			)
 		)
-		(property "LCSC" "C1525"
+		(property "MFR_NUM" "CL05B104KO5NNNC"
 			(at 265.43 114.3 0)
 			(effects
@@
 			)
 		)
-		(property "Value" "MHPA1010RGBDT"
+		(property "Value" "L201DS-QEPGBG2S"
 			(at 222.25 33.145 90)
 			(effects
@@
 			)
 		)
-		(property "Footprint" "Philly_Lib:LED-ARRAY-SMD_4P-L1.0-W1.0-TR-RD"
+		(property "Footprint" "Philly_Lib:L201DS-QEPGBG2S"
 			(at 203.2 30.48 0)
 			(effects
@@
 			)
 		)
-		(property "Datasheet" "https://lcsc.com/product-detail/Light-Emitting-Diodes-LED_MEIHUA-MHPA1010RGBDT_C404280.html"
+		(property "Datasheet" ""
 			(at 200.66 30.48 0)
 			(effects
@@
 			)
 		)
-		(property "LCSC Part" "C404280"
-			(at 198.12 30.48 0)
-			(effects
-				(font
-					(size 1.27 1.27)
-				)
-				(hide yes)
-			)
-		)
 		(property "Note" "Up Firing USER"
 			(at 222.25 33.02 90)
@@
 		(dnp no)
 		(fields_autoplaced yes)
-		(property "Reference" "D1"
+		(property "Reference" "D4"
 			(at 29.21 13.97 0)
 			(effects
@@
 			)
 		)
-		(property "Value" "LESD5D5_0CT1G"
+		(property "Value" "ESD5Z5.0C"
 			(at 29.21 16.51 0)
 			(effects
@@
 			)
 		)
-		(property "LCSC" "C383211"
+		(property "MFR_NUM" "ESD5Z5.0C"
 			(at 29.21 5.08 0)
 			(effects
@@
 			(project "Philly_Node"
 				(path "/14b26dc5-70cb-4d13-ac9b-7e033bbb860b"
-					(reference "D1")
+					(reference "D4")
 					(unit 1)
 				)
@@
 		(on_board yes)
 		(dnp no)
-		(property "Reference" "BAT1"
+		(property "Reference" "SOL1"
 			(at 144.78 182.88 0)
 			(effects
@@
 			)
 		)
-		(property "LCSC" "C968533"
+		(property "MF_NUM" "S2B-PH-SM4-TB(LF)(SN)"
 			(at 144.78 182.88 0)
 			(effects
@@
 			(project "Philly_Node"
 				(path "/14b26dc5-70cb-4d13-ac9b-7e033bbb860b"
-					(reference "BAT1")
+					(reference "SOL1")
 					(unit 1)
 				)
@@
 			)
 		)
-		(property "LCSC" "C1525"
+		(property "MFR_NUM" "CL05B104KO5NNNC"
 			(at 78.74 184.15 0)
 			(effects
@@
 			)
 		)
-		(property "LCSC" "C1547"
+		(property "MFR_NUM" "CC0402JPNPO9BN120"
 			(at 171.45 57.15 90)
 			(effects
@@
 			)
 		)
+		(property "MFR_NUM" "GSB1C41110SSHR"
+			(at 27.94 91.44 0)
+			(effects
+				(font
+					(size 1.27 1.27)
+				)
+				(hide yes)
+			)
+		)
+		(property "MFR" "Amphenol"
+			(at 27.94 91.44 0)
+			(effects
+				(font
+					(size 1.27 1.27)
+				)
+				(hide yes)
+			)
+		)
 		(pin "A12"
 		)
@@
 			)
 		)
-		(property "LCSC" "C1525"
+		(property "MFR_NUM" "CL05B104KO5NNNC"
 			(at 52.07 68.58 0)
 			(effects
@@
 			)
 		)
+		(property "MFR_NUM" "FC3215AN 32.768K-C5NN60KC5"
+			(at 154.94 62.23 90)
+			(effects
+				(font
+					(size 1.27 1.27)
+				)
+				(hide yes)
+			)
+		)
+		(property "MFR" "Epson"
+			(at 154.94 62.23 90)
+			(effects
+				(font
+					(size 1.27 1.27)
+				)
+				(hide yes)
+			)
+		)
 		(pin "2"
 		)
@@
 			)
 		)
-		(property "LCSC" "C47647"
+		(property "MF_NUM" "S2B-PH-SM4-TB(LF)(SN)"
 			(at 15.24 130.81 0)
 			(effects
@@
 			)
 		)
+		(property "MFR" "JST"
+			(at 21.59 132.08 0)
+			(effects
+				(font
+					(size 1.27 1.27)
+				)
+				(hide yes)
+			)
+		)
 		(pin "1"
 		)
@@
 			)
 		)
-		(property "LCSC" "C1525"
+		(property "MFR_NUM" "CL05B104KO5NNNC"
 			(at 171.45 96.52 0)
 			(effects
@@
 		(dnp no)
 		(fields_autoplaced yes)
-		(property "Reference" "D3"
+		(property "Reference" "D4"
 			(at 29.21 34.29 0)
 			(effects
@@
 			)
 		)
-		(property "Value" "LESD5D5_0CT1G"
+		(property "Value" "ESD5Z5.0C"
 			(at 29.21 36.83 0)
 			(effects
@@
 			)
 		)
-		(property "LCSC" "C383211"
+		(property "MFR_NUM" "ESD5Z5.0C"
 			(at 29.21 25.4 0)
 			(effects
@@
 			(project "Philly_Node"
 				(path "/14b26dc5-70cb-4d13-ac9b-7e033bbb860b"
-					(reference "D3")
+					(reference "D4")
 					(unit 1)
 				)
